File: squawkbox_m_0.1.brd (EAGLE design)
At the start: 56.8 x 40.6 mm, 19 parts, among them J2 1X2-3.5MM, U2 RJ45, X3 JSTPH

Commit message: update
Parts:
- flipped R4 to the top
Routing:
- net VCC: track 87.0 -> 101.9 mm, vias 1 -> 3
- net GND: track 147.2 -> 158.8 mm, vias 2 -> 3
- net A4_SDA: track 66.7 -> 55.6 mm, vias 0 -> 1
- net A5_SCL: track 53.8 -> 62.7 mm
- net D5: track 45.4 -> 53.3 mm
- net D4: track 59.9 -> 65.4 mm
- net D8: track 37.2 -> 34.3 mm, vias 2 -> 0
- net D2: track 44.4 -> 41.7 mm
- net PWR: track 100.5 -> 100.3 mm, vias 0 -> 1
